Commit message: correct agv config

File: noovelia_forklift_description/urdf/robot.xacro (robot description, xacro)
@@ -16,13 +16,13 @@
 <link name="chassis_link">
     <collision name="chassis_collision">
-      <origin rpy="0 0 0" xyz="0 0 0"/>
+      <origin rpy="${M_PI_2} 0 0" xyz="0 0 0"/>
         <geometry>
-            <mesh filename="package://noovelia_forklift_description/meshes/Forklift model/carrosserie lift.STL" scale="0.001 0.001 0.001"/>
+            <mesh filename="package://noovelia_forklift_description/meshes/Forklift model/Assemblage général.STL" scale="0.001 0.001 0.001"/>
         </geometry>
     </collision>
     <visual name="chassis_visual">
-      <origin rpy="0 0 0" xyz="0 0 0"/>
+      <origin rpy="${M_PI_2} 0 0" xyz="0 0 0"/>
       <geometry>
-        <mesh filename="package://noovelia_forklift_description/meshes/Forklift model/carrosserie lift.STL" scale="0.001 0.001 0.001"/>
+        <mesh filename="package://noovelia_forklift_description/meshes/Forklift model/Assemblage général.STL" scale="0.001 0.001 0.001"/>
       </geometry>
       <material name="red"/>

Commit message: add list and chassis in urdf model

File: noovelia_forklift_description/urdf/robot.xacro (robot description, xacro)
@@ -16,15 +16,15 @@
 <link name="chassis_link">
     <collision name="chassis_collision">
-      <origin rpy="${M_PI_2} 0 0" xyz="0 0 0"/>
+      <origin rpy="${M_PI_2} 0 0" xyz="0 1 0"/>
         <geometry>
-            <mesh filename="package://noovelia_forklift_description/meshes/Forklift model/Assemblage général.STL" scale="0.001 0.001 0.001"/>
+            <mesh filename="package://noovelia_forklift_description/meshes/Forklift model/chassis AGV FL.STL" scale="0.001 0.001 0.001"/>
         </geometry>
     </collision>
     <visual name="chassis_visual">
-      <origin rpy="${M_PI_2} 0 0" xyz="0 0 0"/>
+      <origin rpy="${M_PI_2} 0 0" xyz="0 1 0"/>
       <geometry>
-        <mesh filename="package://noovelia_forklift_description/meshes/Forklift model/Assemblage général.STL" scale="0.001 0.001 0.001"/>
+        <mesh filename="package://noovelia_forklift_description/meshes/Forklift model/chassis AGV FL.STL" scale="0.001 0.001 0.001"/>
       </geometry>
-      <material name="red"/>
+      <material name="white"/>
     </visual>
 </link>
@@ -34,3 +34,23 @@
     <child link="chassis_link"/>
 </joint>
+ <link name="lift_link">
+    <collision name="lift_collision">
+      <origin rpy="${M_PI/2} 0 0" xyz="0 0 0"/>
+        <geometry>
+            <mesh filename="package://noovelia_robot_description/meshes/Forklift model/carrosserie lift.STL" scale="0.001 0.001 0.001"/>
+        </geometry>
+    </collision>
+    <visual name="lift_visual">
+      <origin rpy="${M_PI/2} 0 0" xyz="0 0 0"/>
+      <geometry>
+        <mesh filename="package://noovelia_robot_description/meshes/Forklift model/carrosserie lift.STL" scale="0.001 0.001 0.001"/>
+      </geometry>
+      <material name="grey"/>
+    </visual>
+  </link>
+  <joint name="lift_joint" type="fixed">
+    <parent link="chassis_link"/>
+    <child link="lift_link"/>
+    <origin xyz="0.6 -1 0.2"/>
+  </joint>
 </robot>

Commit message: Added some gazebo references and interia

File: noovelia_forklift_description/urdf/robot.xacro (robot description, xacro)
@@ -4,4 +4,11 @@
   <xacro:property name="M_PI_2" value="1.570796327" />
   <xacro:property name="DEG_TO_RAD" value="0.017453293" />
+   <xacro:macro name="default_inertial" params="mass w h d">
+    <inertial>
+      <origin rpy="0 0 0" xyz="${d/2} -${w/2} ${h/2}"/>
+      <mass value="${mass}" />
+      <inertia ixx="${(1/12)*(h*h + d*d)}" ixy="0.0" ixz="0.0" iyy="${(1/12)*(w*w + d*d)}" iyz="0.0" izz="${(1/12)*(w*w + h*h)}" />
+    </inertial>
+  </xacro:macro>
   <xacro:include filename="$(find noovelia_forklift_description)/urdf/material.xacro" />
   <!-- base_footprint is a fictitious link(frame) that is on the ground right below chassis_link origin -->
@@ -28,4 +35,9 @@
       <material name="white"/>
     </visual>
+    <inertial>
+      <origin rpy="0 0 0" xyz="0 0 0"/>
+      <mass value="40" />
+    <inertia ixx="0.1" ixy="0.0" ixz="0.0" iyy="0.1" iyz="0.0" izz="0.1" />
+    </inertial>
 </link>
 <joint name="base_footprint_joint" type="fixed">
@@ -46,6 +58,7 @@
         <mesh filename="package://noovelia_robot_description/meshes/Forklift model/carrosserie lift.STL" scale="0.001 0.001 0.001"/>
       </geometry>
-      <material name="grey"/>
+      <material name="red"/>
     </visual>
+    <xacro:default_inertial mass="40" w = "1.1" h = "1.2" d = "0.9"/>
   </link>
   <joint name="lift_joint" type="fixed">
@@ -54,3 +67,15 @@
     <origin xyz="0.6 -1 0.2"/>
   </joint>
+  <!--gazebo references-->
+   <gazebo reference="base_footprint">
+        <turnGravityOff>false</turnGravityOff>
+    </gazebo>
+    <gazebo reference="chassis_link">
+        <turnGravityOff>false</turnGravityOff>
+        <material>Gazebo/Orange</material>
+    </gazebo>
+    <gazebo reference="lift_link">
+        <turnGravityOff>false</turnGravityOff>
+        <material>Gazebo/Orange</material>
+    </gazebo>
 </robot>

Commit message: added gazebo launch file

File: noovelia_forklift_description/urdf/robot.xacro (robot description, xacro)
@@ -36,5 +36,5 @@
     </visual>
     <inertial>
-      <origin rpy="0 0 0" xyz="0 0 0"/>
+      <origin rpy="0 0 0" xyz="1.1 -0.7 0.3"/>
       <mass value="40" />
     <inertia ixx="0.1" ixy="0.0" ixz="0.0" iyy="0.1" iyz="0.0" izz="0.1" />

Commit message: added main wheel

File: noovelia_forklift_description/urdf/robot.xacro (robot description, xacro)
@@ -4,4 +4,8 @@
   <xacro:property name="M_PI_2" value="1.570796327" />
   <xacro:property name="DEG_TO_RAD" value="0.017453293" />
+  <!--the main wheel that perform steer + move behind the lift-->
+  <xacro:property name="wheel_width" value="0.2" />
+  <xacro:property name="wheel_radius" value="0.225" />
+  <xacro:property name="wheel_mass" value="4" /> <!-- in kg-->
    <xacro:macro name="default_inertial" params="mass w h d">
     <inertial>
@@ -11,5 +15,11 @@
     </inertial>
   </xacro:macro>
+  <xacro:macro name="cylinder_inertia" params="m r h">
+      <inertia  ixx="${m*(3*r*r+h*h)/12}" ixy = "0" ixz = "0"
+                iyy="${m*(3*r*r+h*h)/12}" iyz = "0"
+                izz="${m*r*r/2}" />
+  </xacro:macro>
   <xacro:include filename="$(find noovelia_forklift_description)/urdf/material.xacro" />
+  <xacro:include filename="$(find noovelia_forklift_description)/urdf/wheel.xacro" />
   <!-- base_footprint is a fictitious link(frame) that is on the ground right below chassis_link origin -->
   <link name="base_footprint">
@@ -23,5 +33,5 @@
 <link name="chassis_link">
     <collision name="chassis_collision">
-      <origin rpy="${M_PI_2} 0 0" xyz="0 1 0"/>
+      <origin rpy="${M_PI_2} 0 0" xyz="0 1 -0.2"/>
         <geometry>
             <mesh filename="package://noovelia_forklift_description/meshes/Forklift model/chassis AGV FL.STL" scale="0.001 0.001 0.001"/>
@@ -29,5 +39,5 @@
     </collision>
     <visual name="chassis_visual">
-      <origin rpy="${M_PI_2} 0 0" xyz="0 1 0"/>
+      <origin rpy="${M_PI_2} 0 0" xyz="0 1 -0.2"/>
       <geometry>
         <mesh filename="package://noovelia_forklift_description/meshes/Forklift model/chassis AGV FL.STL" scale="0.001 0.001 0.001"/>
@@ -65,6 +75,11 @@
     <parent link="chassis_link"/>
     <child link="lift_link"/>
-    <origin xyz="0.6 -1 0.2"/>
+    <origin xyz="0.6 -1 0.15"/>
   </joint>
+  <!--main wheel-->
+  <xacro:wheel_link prefix="wheel" mesh = "package://noovelia_robot_description/meshes/Forklift model/Moteur MV300.STL"
+                  mass= "${wheel_mass}" radius= "${wheel_radius}"
+                  width= "${wheel_width}" origin_rpy="0 0 0"/>
+  <xacro:wheel_joint prefix="wheel" child = "wheel_link" origin_xyz = "1.05 -1.7 0"/>
   <!--gazebo references-->
    <gazebo reference="base_footprint">

Commit message: added gaebo reference

File: noovelia_forklift_description/urdf/robot.xacro (robot description, xacro)
@@ -94,3 +94,12 @@
         <material>Gazebo/Orange</material>
     </gazebo>
+    <gazebo reference="wheel_link">
+        <mu1 value="1.0"/>
+        <mu2 value="1.0"/>
+        <kp  value="10000.0" />
+        <kd  value="1.0" />
+        <fdir1 value="1 0 0"/>
+        <material>Gazebo/Grey</material>
+        <turnGravityOff>false</turnGravityOff>
+    </gazebo>
 </robot>
