Commit message: Added links for steer and movegit add .

File: forklift_description/urdf/robot.xacro (robot description, xacro)
@@ -22,5 +22,5 @@
   <xacro:include filename="$(find forklift_description)/urdf/material.xacro" />
   <xacro:include filename="$(find forklift_description)/urdf/wheel.xacro" />
-  <!-- base_footprint is a fictitious link(frame) that is on the ground right below chassis_link origin -->
+  <!-- base_footprint is a fictitious link(frame) that is on the ground right below base_fork origin -->
   <link name="base_footprint">
     <visual>
@@ -31,13 +31,13 @@
     </visual>
   </link>>
-<link name="chassis_link">
-    <collision name="chassis_collision">
-      <origin rpy="${M_PI_2} 0 0" xyz="0 1 -0.2"/>
+<link name="base_fork">
+    <collision name="fork_collision">
+      <origin rpy="${M_PI_2} 0 0" xyz="-1.25 0.8 -0.2"/>
         <geometry>
             <mesh filename="package://forklift_description/meshes/Forklift model/chassis AGV FL.STL" scale="0.001 0.001 0.001"/>
         </geometry>
     </collision>
-    <visual name="chassis_visual">
-      <origin rpy="${M_PI_2} 0 0" xyz="0 1 -0.2"/>
+    <visual name="fork_visual">
+      <origin rpy="${M_PI_2} 0 0" xyz="-1.25 0.8 -0.2"/>
       <geometry>
         <mesh filename="package://forklift_description/meshes/Forklift model/chassis AGV FL.STL" scale="0.001 0.001 0.001"/>
@@ -51,18 +51,18 @@
     </inertial>
 </link>
-<joint name="base_footprint_joint" type="fixed">
-    <origin rpy="0 0 0" xyz="0 0 0"/>
+<joint name="base_fork_joint" type="fixed">
+    <origin rpy="0 0 0" xyz="0 0.25 0"/>
     <parent link="base_footprint"/>
-    <child link="chassis_link"/>
+    <child link="base_fork"/>
 </joint>
- <link name="lift_link">
-    <collision name="lift_collision">
-      <origin rpy="${M_PI/2} 0 0" xyz="0 0 0"/>
+ <link name="base_link">
+    <collision name="base_link_collision">
+      <origin rpy="${M_PI/2} 0 0" xyz="-0.6 -1.1 0"/>
         <geometry>
             <mesh filename="package://noovelia_robot_description/meshes/Forklift model/carrosserie lift.STL" scale="0.001 0.001 0.001"/>
         </geometry>
     </collision>
-    <visual name="lift_visual">
-      <origin rpy="${M_PI/2} 0 0" xyz="0 0 0"/>
+    <visual name="base_link_visual">
+      <origin rpy="${M_PI/2} 0 0" xyz="-0.6 -1.1 0"/>
       <geometry>
         <mesh filename="package://noovelia_robot_description/meshes/Forklift model/carrosserie lift.STL" scale="0.001 0.001 0.001"/>
@@ -72,34 +72,68 @@
     <xacro:default_inertial mass="40" w = "1.1" h = "1.2" d = "0.9"/>
   </link>
-  <joint name="lift_joint" type="fixed">
-    <parent link="chassis_link"/>
-    <child link="lift_link"/>
-    <origin xyz="0.6 -1 0.15"/>
+  <joint name="base_link_joint" type="fixed">
+    <parent link="base_fork"/>
+    <child link="base_link"/>
+    <origin xyz="0 0 0.08"/>
   </joint>
-  <!--main wheel-->
-  <xacro:wheel_link prefix="wheel" mesh = "package://noovelia_robot_description/meshes/Forklift model/Moteur MV300.STL"
-                  mass= "${wheel_mass}" radius= "${wheel_radius}"
-                  width= "${wheel_width}" origin_rpy="0 0 0"/>
-  <xacro:wheel_joint prefix="wheel" child = "wheel_link" origin_xyz = "1.05 -1.7 0"/>
+      <link name="steer_link">
+        <inertial>
+          <mass value="0.01"/>
+          <inertia ixx="0.001" ixy="0" ixz="0" iyy="0.001" iyz="0" izz="0.001" />
+          <origin/>
+        </inertial>
+        <visual>
+          <origin xyz="0 0 0" rpy="0 0 0" />
+          <geometry>
+            <box size="0.2 0.2 0.2" />
+          </geometry>
+          <material name="orange"/>
+        </visual>
+      </link>
+      <link name="sd_wheel_link">
+        <inertial>
+          <mass value="10"/>
+          <inertia ixx="0.01" ixy="0" ixz="0" iyy="0.01" iyz="0" izz="0.01" />
+          <origin/>
+        </inertial>
+        <visual>
+          <origin xyz="0 0 0" rpy="${M_PI_2} 0 ${M_PI_2}" />
+          <geometry>
+            <cylinder radius="0.16" length="0.04" />
+          </geometry>
+          <material name="black"/>
+        </visual>
+        <collision>
+          <origin xyz="0 0 0" rpy="${M_PI_2} 0 ${M_PI_2}" />
+          <geometry>
+            <cylinder radius="0.16" length="0.04" />
+          </geometry>
+        </collision>
+      </link>
+      <joint name="base2steer_joint" type="revolute">
+        <parent link="base_link"/>
+        <child link="steer_link"/>
+        <limit effort="10000.0" lower="-${M_PI_2}" upper="${M_PI_2}" velocity="100"/>
+        <origin xyz="0 -1.6 0.05" rpy="0 0 0" />
+        <axis xyz="0 0 1" />
+      </joint>
+      <joint name="steer2sd_wheel_joint" type="continuous">
+        <parent link="steer_link"/>
+        <child link="sd_wheel_link"/>
+        <limit effort="10000.0" velocity="100"/>
+        <origin xyz="0 0 0" rpy="0 0 0" />
+        <axis xyz="0 1 0" />
+      </joint>
   <!--gazebo references-->
    <gazebo reference="base_footprint">
         <turnGravityOff>false</turnGravityOff>
     </gazebo>
-    <gazebo reference="chassis_link">
+    <gazebo reference="base_fork">
         <turnGravityOff>false</turnGravityOff>
         <material>Gazebo/Orange</material>
     </gazebo>
-    <gazebo reference="lift_link">
+    <gazebo reference="base_link">
         <turnGravityOff>false</turnGravityOff>
         <material>Gazebo/Orange</material>
     </gazebo>
-    <gazebo reference="wheel_link">
-        <mu1 value="1.0"/>
-        <mu2 value="1.0"/>
-        <kp  value="10000.0" />
-        <kd  value="1.0" />
-        <fdir1 value="1 0 0"/>
-        <material>Gazebo/Grey</material>
-        <turnGravityOff>false</turnGravityOff>
-    </gazebo>
 </robot>

Commit message: Place the main wheel in right position

File: forklift_description/urdf/robot.xacro (robot description, xacro)
@@ -5,6 +5,6 @@
   <xacro:property name="DEG_TO_RAD" value="0.017453293" />
   <!--the main wheel that perform steer + move behind the lift-->
-  <xacro:property name="wheel_width" value="0.2" />
-  <xacro:property name="wheel_radius" value="0.225" />
+  <xacro:property name="wheel_width" value="0.06" />
+  <xacro:property name="wheel_radius" value="0.12" />
   <xacro:property name="wheel_mass" value="4" /> <!-- in kg-->
    <xacro:macro name="default_inertial" params="mass w h d">
@@ -21,5 +21,4 @@
   </xacro:macro>
   <xacro:include filename="$(find forklift_description)/urdf/material.xacro" />
-  <xacro:include filename="$(find forklift_description)/urdf/wheel.xacro" />
   <!-- base_footprint is a fictitious link(frame) that is on the ground right below base_fork origin -->
   <link name="base_footprint">
@@ -58,5 +57,5 @@
  <link name="base_link">
     <collision name="base_link_collision">
-      <origin rpy="${M_PI/2} 0 0" xyz="-0.6 -1.1 0"/>
+      <origin rpy="${M_PI/2} 0 0" xyz="-0.6 -1.1 -${wheel_radius}"/>
         <geometry>
             <mesh filename="package://noovelia_robot_description/meshes/Forklift model/carrosserie lift.STL" scale="0.001 0.001 0.001"/>
@@ -64,5 +63,5 @@
     </collision>
     <visual name="base_link_visual">
-      <origin rpy="${M_PI/2} 0 0" xyz="-0.6 -1.1 0"/>
+      <origin rpy="${M_PI/2} 0 0" xyz="-0.6 -1.1 -${wheel_radius}"/>
       <geometry>
         <mesh filename="package://noovelia_robot_description/meshes/Forklift model/carrosserie lift.STL" scale="0.001 0.001 0.001"/>
@@ -75,5 +74,5 @@
     <parent link="base_fork"/>
     <child link="base_link"/>
-    <origin xyz="0 0 0.08"/>
+    <origin xyz="0 0 ${wheel_radius}"/>
   </joint>
       <link name="steer_link">
@@ -86,5 +85,5 @@
           <origin xyz="0 0 0" rpy="0 0 0" />
           <geometry>
-            <box size="0.2 0.2 0.2" />
+            <box size="0.16 0.16 0.16" />
           </geometry>
           <material name="orange"/>
@@ -100,5 +99,5 @@
           <origin xyz="0 0 0" rpy="${M_PI_2} 0 ${M_PI_2}" />
           <geometry>
-            <cylinder radius="0.16" length="0.04" />
+            <cylinder radius="${wheel_radius}" length="${wheel_width}" />
           </geometry>
           <material name="black"/>
@@ -107,5 +106,5 @@
           <origin xyz="0 0 0" rpy="${M_PI_2} 0 ${M_PI_2}" />
           <geometry>
-            <cylinder radius="0.16" length="0.04" />
+            <cylinder radius="${wheel_radius}" length="${wheel_width}" />
           </geometry>
         </collision>
@@ -115,5 +114,5 @@
         <child link="steer_link"/>
         <limit effort="10000.0" lower="-${M_PI_2}" upper="${M_PI_2}" velocity="100"/>
-        <origin xyz="0 -1.6 0.05" rpy="0 0 0" />
+        <origin xyz="0 -1.6 0" rpy="0 0 0" />
         <axis xyz="0 0 1" />
       </joint>

Commit message: added support wheels

File: forklift_description/urdf/robot.xacro (robot description, xacro)
@@ -124,4 +124,56 @@
         <axis xyz="0 1 0" />
       </joint>
+      <link name="fixed_left_wheel_link">
+        <inertial>
+          <mass value="0.1"/>
+          <inertia ixx="0.01" ixy="0" ixz="0" iyy="0.01" iyz="0" izz="0.01" />
+          <origin/>
+        </inertial>
+        <visual>
+          <origin xyz="0 0.11 0" rpy="1.57 0 0" />
+          <geometry>
+            <mesh filename="package://noovelia_robot_description/meshes/Forklift model/Roues avant.STL" scale="0.001 0.001 0.001"/>
+          </geometry>
+          <material name="grey"/>
+        </visual>
+        <collision>
+          <origin xyz="0 0.11 0" rpy="1.57 0 0" />
+          <geometry>
+            <mesh filename="package://noovelia_robot_description/meshes/Forklift model/Roues avant.STL" scale="0.001 0.001 0.001"/>
+          </geometry>
+         <!-- <contact_coefficients mu="100" kp="10.0" kd="0.1"/> -->
+        </collision>
+      </link>
+      <joint name="base2fixed_left_wheel_joint" type="fixed">
+        <parent link="base_fork"/>
+        <child link="fixed_left_wheel_link"/>
+        <origin xyz="0.45 0.05 0.03" rpy="0 0 0" />
+      </joint>
+      <link name="fixed_right_wheel_link">
+        <inertial>
+          <mass value="0.1"/>
+          <inertia ixx="0.01" ixy="0" ixz="0" iyy="0.01" iyz="0" izz="0.01" />
+          <origin/>
+        </inertial>
+        <visual>
+          <origin xyz="0 0.11 0" rpy="1.57 0 0" />
+          <geometry>
+            <mesh filename="package://noovelia_robot_description/meshes/Forklift model/Roues avant.STL" scale="0.001 0.001 0.001"/>
+          </geometry>
+          <material name="grey"/>
+        </visual>
+        <collision>
+          <origin xyz="0 0.11 0" rpy="1.57 0 0" />
+          <geometry>
+            <mesh filename="package://noovelia_robot_description/meshes/Forklift model/Roues avant.STL" scale="0.001 0.001 0.001"/>
+          </geometry>
+         <!-- <contact_coefficients mu="100" kp="10.0" kd="0.1"/> -->
+        </collision>
+      </link>
+      <joint name="base2fixed_right_wheel_joint" type="fixed">
+        <parent link="base_fork"/>
+        <child link="fixed_right_wheel_link"/>
+        <origin xyz="-0.6 0.05 0.03" rpy="0 0 0" />
+      </joint>
   <!--gazebo references-->
    <gazebo reference="base_footprint">

Commit message: add gazebo references

File: forklift_description/urdf/robot.xacro (robot description, xacro)
@@ -8,7 +8,7 @@
   <xacro:property name="wheel_radius" value="0.12" />
   <xacro:property name="wheel_mass" value="4" /> <!-- in kg-->
-   <xacro:macro name="default_inertial" params="mass w h d">
+   <xacro:macro name="default_inertial" params="mass w h d yorigin">
     <inertial>
-      <origin rpy="0 0 0" xyz="${d/2} -${w/2} ${h/2}"/>
+      <origin rpy="0 0 0" xyz="0 -${yorigin} ${h/2}"/>
       <mass value="${mass}" />
       <inertia ixx="${(1/12)*(h*h + d*d)}" ixy="0.0" ixz="0.0" iyy="${(1/12)*(w*w + d*d)}" iyz="0.0" izz="${(1/12)*(w*w + h*h)}" />
@@ -45,5 +45,5 @@
     </visual>
     <inertial>
-      <origin rpy="0 0 0" xyz="1.1 -0.7 0.3"/>
+      <origin rpy="0 0 0" xyz="0 -0.7 0.3"/>
       <mass value="40" />
     <inertia ixx="0.1" ixy="0.0" ixz="0.0" iyy="0.1" iyz="0.0" izz="0.1" />
@@ -69,5 +69,5 @@
       <material name="red"/>
     </visual>
-    <xacro:default_inertial mass="40" w = "1.1" h = "1.2" d = "0.9"/>
+    <xacro:default_inertial mass="40" w = "1.1" h = "1.2" d = "0.9" yorigin = "1.6"/>
   </link>
   <joint name="base_link_joint" type="fixed">
@@ -188,3 +188,25 @@
         <material>Gazebo/Orange</material>
     </gazebo>
+    <gazebo reference="steer_link">
+      <material>Gazebo/Orange</material>
+    </gazebo>
+    <gazebo reference="fixed_left_wheel_link" >
+      <material>Gazebo/Black</material>
+    </gazebo>
+    <gazebo reference="fixed_right_wheel_link" >
+      <material>Gazebo/Black</material>
+    </gazebo>
+    <gazebo reference="sd_wheel_link" >
+    <!-- <mu1 value="10000.0" />
+    <mu2 value="10000.0" />
+    <kp  value="10000000000.0" />
+    <kd  value="1.0" /> -->
+      <material>Gazebo/Black</material>
+  </gazebo>
+      <!-- ros_control plugin -->
+  <gazebo>
+    <plugin name="gazebo_ros_control" filename="libgazebo_ros_control.so">
+<!--      <robotNamespace>/forklift</robotNamespace> -->
+    </plugin>
+  </gazebo>
 </robot>

Commit message: Make extra wheel continous only used for tf

File: forklift_description/urdf/robot.xacro (robot description, xacro)
@@ -145,8 +145,9 @@
         </collision>
       </link>
-      <joint name="base2fixed_left_wheel_joint" type="fixed">
+      <joint name="base2fixed_left_wheel_joint" type="continuous">
         <parent link="base_fork"/>
         <child link="fixed_left_wheel_link"/>
         <origin xyz="0.45 0.05 0.03" rpy="0 0 0" />
+        <axis xyz="0 1 0" />
       </joint>
       <link name="fixed_right_wheel_link">
@@ -171,8 +172,9 @@
         </collision>
       </link>
-      <joint name="base2fixed_right_wheel_joint" type="fixed">
+      <joint name="base2fixed_right_wheel_joint" type="continuous">
         <parent link="base_fork"/>
         <child link="fixed_right_wheel_link"/>
         <origin xyz="-0.6 0.05 0.03" rpy="0 0 0" />
+        <axis xyz="0 1 0" />
       </joint>
   <!--gazebo references-->
@@ -198,8 +200,8 @@
     </gazebo>
     <gazebo reference="sd_wheel_link" >
-    <!-- <mu1 value="10000.0" />
+    <mu1 value="10000.0" />
     <mu2 value="10000.0" />
     <kp  value="10000000000.0" />
-    <kd  value="1.0" /> -->
+    <kd  value="1.0" />
       <material>Gazebo/Black</material>
   </gazebo>
@@ -210,3 +212,25 @@
     </plugin>
   </gazebo>
+   <gazebo>
+    <plugin name="steer_drive_controller" filename="libgazebo_ros_steer_drive.so">
+      <alwaysOn>true</alwaysOn>
+      <updateRate>100</updateRate>
+      <steerJoint>base2steer_joint</steerJoint>
+      <driveJoint>steer2sd_wheel_joint</driveJoint>
+      <fixedWheelLeftJoint>base2fixed_left_wheel_joint</fixedWheelLeftJoint>
+      <fixedWheelRightJoint>base2fixed_right_wheel_joint</fixedWheelRightJoint>
+      <wheelDiameter>${2*wheel_radius}</wheelDiameter>
+      <steeringFixWheelDistanceX>1.190</steeringFixWheelDistanceX>
+      <steeringFixWheelDistanceY>0.0</steeringFixWheelDistanceY>
+      <steerTorque>1000</steerTorque>
+      <driveTorque>1000</driveTorque>
+      <commandTopic>cmd_vel</commandTopic>
+      <odometryTopic>odom</odometryTopic>
+      <odometryFrame>/world</odometryFrame>
+      <robotBaseFrame>base_footprint</robotBaseFrame>
+      <odomEncSteeringAngleOffset>0.01</odomEncSteeringAngleOffset>
+      <!--odometrySource>encoder</odometrySource-->
+      <publishWheelJointState>true</publishWheelJointState>
+    </plugin>
+  </gazebo>
 </robot>

Commit message: correct axis of rotation for the wheels

File: forklift_description/urdf/robot.xacro (robot description, xacro)
@@ -7,5 +7,5 @@
   <xacro:property name="wheel_width" value="0.06" />
   <xacro:property name="wheel_radius" value="0.12" />
-  <xacro:property name="wheel_mass" value="4" /> <!-- in kg-->
+  <xacro:property name="wheel_mass" value="10" /> <!-- in kg-->
    <xacro:macro name="default_inertial" params="mass w h d yorigin">
     <inertial>
@@ -78,5 +78,5 @@
       <link name="steer_link">
         <inertial>
-          <mass value="0.01"/>
+          <mass value="0.05"/>
           <inertia ixx="0.001" ixy="0" ixz="0" iyy="0.001" iyz="0" izz="0.001" />
           <origin/>
@@ -92,5 +92,5 @@
       <link name="sd_wheel_link">
         <inertial>
-          <mass value="10"/>
+          <mass value="${wheel_mass}"/>
           <inertia ixx="0.01" ixy="0" ixz="0" iyy="0.01" iyz="0" izz="0.01" />
           <origin/>
@@ -122,5 +122,5 @@
         <limit effort="10000.0" velocity="100"/>
         <origin xyz="0 0 0" rpy="0 0 0" />
-        <axis xyz="0 1 0" />
+        <axis xyz="1 0 0" />
       </joint>
       <link name="fixed_left_wheel_link">
@@ -148,6 +148,6 @@
         <parent link="base_fork"/>
         <child link="fixed_left_wheel_link"/>
-        <origin xyz="0.45 0.05 0.03" rpy="0 0 0" />
-        <axis xyz="0 1 0" />
+        <origin xyz="0.45 0.05 0.02" rpy="0 0 0" />
+        <axis xyz="1 0 0" />
       </joint>
       <link name="fixed_right_wheel_link">
@@ -175,6 +175,6 @@
         <parent link="base_fork"/>
         <child link="fixed_right_wheel_link"/>
-        <origin xyz="-0.6 0.05 0.03" rpy="0 0 0" />
-        <axis xyz="0 1 0" />
+        <origin xyz="-0.6 0.05 0.02" rpy="0 0 0" />
+        <axis xyz="1 0 0" />
       </joint>
   <!--gazebo references-->

Commit message: correct inertia

File: forklift_description/urdf/robot.xacro (robot description, xacro)
@@ -45,5 +45,5 @@
     </visual>
     <inertial>
-      <origin rpy="0 0 0" xyz="0 -0.7 0.3"/>
+      <origin rpy="0 0 0" xyz="0 -0.2 0.3"/>
       <mass value="40" />
     <inertia ixx="0.1" ixy="0.0" ixz="0.0" iyy="0.1" iyz="0.0" izz="0.1" />
@@ -229,5 +229,5 @@
       <odometryFrame>/world</odometryFrame>
       <robotBaseFrame>base_footprint</robotBaseFrame>
-      <wheelAcceleration>1</wheelAcceleration>
+      <wheelAcceleration>0.5</wheelAcceleration>
       <odomEncSteeringAngleOffset>0.01</odomEncSteeringAngleOffset>
       <!--odometrySource>encoder</odometrySource-->

Commit message: change some gazebo coeff

File: forklift_description/urdf/robot.xacro (robot description, xacro)
@@ -3,4 +3,5 @@
   <xacro:property name="M_PI" value="3.1415926535897931" />
   <xacro:property name="M_PI_2" value="1.570796327" />
+  <xacro:property name="M_PI_4" value="0.785" />
   <xacro:property name="DEG_TO_RAD" value="0.017453293" />
   <!--the main wheel that perform steer + move behind the lift-->
@@ -45,5 +46,5 @@
     </visual>
     <inertial>
-      <origin rpy="0 0 0" xyz="0 -0.2 0.3"/>
+      <origin rpy="0 0 0" xyz="0 -0.1 0.4"/>
       <mass value="40" />
     <inertia ixx="0.1" ixy="0.0" ixz="0.0" iyy="0.1" iyz="0.0" izz="0.1" />
@@ -113,6 +114,6 @@
         <parent link="base_link"/>
         <child link="steer_link"/>
-        <limit effort="10000.0" lower="-${M_PI_2}" upper="${M_PI_2}" velocity="100"/>
-        <origin xyz="0 -1.6 0" rpy="0 0 0" />
+        <limit effort="10000.0" lower="-${M_PI_4}" upper="${M_PI_4}" velocity="100"/>
+        <origin xyz="0 -1.7 0" rpy="0 0 0" />
         <axis xyz="0 0 1" />
       </joint>
@@ -194,15 +195,23 @@
     </gazebo>
     <gazebo reference="fixed_left_wheel_link" >
+      <mu1 value="10000.0" />
+      <mu2 value="10000.0" />
+      <kp  value="10000000000.0" />
+      <kd  value="1.0" />
       <material>Gazebo/Black</material>
     </gazebo>
     <gazebo reference="fixed_right_wheel_link" >
+      <mu1 value="10000.0" />
+      <mu2 value="10000.0" />
+      <kp  value="10000000000.0" />
+      <kd  value="1.0" />
       <material>Gazebo/Black</material>
     </gazebo>
     <gazebo reference="sd_wheel_link" >
-    <mu1 value="10000.0" />
-    <mu2 value="10000.0" />
-    <kp  value="10000000000.0" />
-    <kd  value="1.0" />
-      <material>Gazebo/Black</material>
+      <mu1 value="10000.0" />
+      <mu2 value="10000.0" />
+      <kp  value="10000000000.0" />
+      <kd  value="1.0" />
+    <material>Gazebo/Black</material>
   </gazebo>
       <!-- ros_control plugin -->
