Commit message: xacro changes

File: forklift_description/urdf/robot.xacro (robot description, xacro)
@@ -6,5 +6,5 @@
   <xacro:property name="DEG_TO_RAD" value="0.017453293" />
   <!--the main wheel that perform steer + move behind the lift-->
-  <xacro:property name="wheel_width" value="0.06" />
+  <xacro:property name="wheel_width" value="0.09" />
   <xacro:property name="wheel_radius" value="0.12" />
   <xacro:property name="wheel_mass" value="10" /> <!-- in kg-->
@@ -46,5 +46,5 @@
     </visual>
     <inertial>
-      <origin rpy="0 0 0" xyz="0 -0.1 0.4"/>
+      <origin rpy="0 0 0" xyz="0 -0.2 0.3"/>
       <mass value="40" />
     <inertia ixx="0.1" ixy="0.0" ixz="0.0" iyy="0.1" iyz="0.0" izz="0.1" />
@@ -114,6 +114,6 @@
         <parent link="base_link"/>
         <child link="steer_link"/>
-        <limit effort="10000.0" lower="-${M_PI_4}" upper="${M_PI_4}" velocity="100"/>
-        <origin xyz="0 -1.7 0" rpy="0 0 0" />
+        <limit effort="10000.0" lower="-${M_PI_2}" upper="${M_PI_2}" velocity="100"/>
+        <origin xyz="0 -1.65 0" rpy="0 0 0" />
         <axis xyz="0 0 1" />
       </joint>
@@ -146,9 +146,9 @@
         </collision>
       </link>
-      <joint name="base2fixed_left_wheel_joint" type="continuous">
+      <joint name="base2fixed_left_wheel_joint" type="fixed">
         <parent link="base_fork"/>
         <child link="fixed_left_wheel_link"/>
         <origin xyz="0.45 0.05 0.02" rpy="0 0 0" />
-        <axis xyz="1 0 0" />
+        <!-- <axis xyz="1 0 0" /> -->
       </joint>
       <link name="fixed_right_wheel_link">
@@ -173,9 +173,9 @@
         </collision>
       </link>
-      <joint name="base2fixed_right_wheel_joint" type="continuous">
+      <joint name="base2fixed_right_wheel_joint" type="fixed">
         <parent link="base_fork"/>
         <child link="fixed_right_wheel_link"/>
         <origin xyz="-0.6 0.05 0.02" rpy="0 0 0" />
-        <axis xyz="1 0 0" />
+        <!-- <axis xyz="1 0 0" /> -->
       </joint>
   <!--gazebo references-->
@@ -192,18 +192,18 @@
     </gazebo>
     <gazebo reference="steer_link">
-      <material>Gazebo/Orange</material>
+      <material>Gazebo/Blue</material>
     </gazebo>
     <gazebo reference="fixed_left_wheel_link" >
-      <mu1 value="10000.0" />
+      <!-- <mu1 value="10000.0" />
       <mu2 value="10000.0" />
       <kp  value="10000000000.0" />
-      <kd  value="1.0" />
+      <kd  value="1.0" /> -->
       <material>Gazebo/Black</material>
     </gazebo>
     <gazebo reference="fixed_right_wheel_link" >
-      <mu1 value="10000.0" />
+      <!-- <mu1 value="10000.0" />
       <mu2 value="10000.0" />
       <kp  value="10000000000.0" />
-      <kd  value="1.0" />
+      <kd  value="1.0" /> -->
       <material>Gazebo/Black</material>
     </gazebo>
@@ -227,6 +227,6 @@
       <steerJoint>base2steer_joint</steerJoint>
       <driveJoint>steer2sd_wheel_joint</driveJoint>
-      <fixedWheelLeftJoint>base2fixed_left_wheel_joint</fixedWheelLeftJoint>
-      <fixedWheelRightJoint>base2fixed_right_wheel_joint</fixedWheelRightJoint>
+      <!-- <fixedWheelLeftJoint>base2fixed_left_wheel_joint</fixedWheelLeftJoint>
+      <fixedWheelRightJoint>base2fixed_right_wheel_joint</fixedWheelRightJoint> -->
       <wheelDiameter>${2*wheel_radius}</wheelDiameter>
       <steeringFixWheelDistanceX>1.190</steeringFixWheelDistanceX>

Commit message: added laser

File: forklift_description/urdf/robot.xacro (robot description, xacro)
@@ -5,4 +5,14 @@
   <xacro:property name="M_PI_4" value="0.785" />
   <xacro:property name="DEG_TO_RAD" value="0.017453293" />
+  <!--laser properties -->
+	<xacro:property name="laserMass" value="0.01"/>
+	<xacro:property name="laserLength" value="0.05"/>
+	<xacro:property name="laserWidth" value="0.05"/>
+	<xacro:property name="laserHeight" value="0.07"/>
+	<xacro:property name="laserOffsetX" value="0"/>
+  <xacro:property name="laserOffsetY" value="-0.7"/>
+	<!--xacro:property name="laserOffsetX" value="0.05"/-->
+	<xacro:property name="laserOffsetZ" value="2.8"/>
+	<!--xacro:property name="laserOffsetZ" value="0.1125"/-->
   <!--the main wheel that perform steer + move behind the lift-->
   <xacro:property name="wheel_width" value="0.09" />
@@ -21,6 +31,12 @@
                 izz="${m*r*r/2}" />
   </xacro:macro>
+  <xacro:macro name="box_inertia" params="m x y z">
+    <inertia  ixx="${m*(y*y+z*z)/12}" ixy = "0" ixz = "0"
+    			iyy="${m*(x*x+z*z)/12}" iyz = "0"
+    			izz="${m*(x*x+z*z)/12}"
+    />
+  </xacro:macro>
   <xacro:include filename="$(find forklift_description)/urdf/material.xacro" />
-  <!-- base_footprint is a fictitious link(frame) that is on the ground right below base_fork origin -->
+<!-- base_footprint is a fictitious link(frame) that is on the ground right below base_link origin, navigation stack dedpends on this frame and KDL needs a root link without any intertia -->
   <link name="base_footprint">
     <visual>
@@ -60,5 +76,5 @@
       <origin rpy="${M_PI/2} 0 0" xyz="-0.6 -1.1 -${wheel_radius}"/>
         <geometry>
-            <mesh filename="package://noovelia_robot_description/meshes/Forklift model/carrosserie lift.STL" scale="0.001 0.001 0.001"/>
+            <mesh filename="package://forklift_description/meshes/Forklift model/carrosserie lift.STL" scale="0.001 0.001 0.001"/>
         </geometry>
     </collision>
@@ -66,5 +82,5 @@
       <origin rpy="${M_PI/2} 0 0" xyz="-0.6 -1.1 -${wheel_radius}"/>
       <geometry>
-        <mesh filename="package://noovelia_robot_description/meshes/Forklift model/carrosserie lift.STL" scale="0.001 0.001 0.001"/>
+        <mesh filename="package://forklift_description/meshes/Forklift model/carrosserie lift.STL" scale="0.001 0.001 0.001"/>
       </geometry>
       <material name="red"/>
@@ -134,5 +150,5 @@
           <origin xyz="0 0.11 0" rpy="1.57 0 0" />
           <geometry>
-            <mesh filename="package://noovelia_robot_description/meshes/Forklift model/Roues avant.STL" scale="0.001 0.001 0.001"/>
+            <mesh filename="package://forklift_description/meshes/Forklift model/Roues avant.STL" scale="0.001 0.001 0.001"/>
           </geometry>
           <material name="grey"/>
@@ -141,5 +157,5 @@
           <origin xyz="0 0.11 0" rpy="1.57 0 0" />
           <geometry>
-            <mesh filename="package://noovelia_robot_description/meshes/Forklift model/Roues avant.STL" scale="0.001 0.001 0.001"/>
+            <mesh filename="package://forklift_description/meshes/Forklift model/Roues avant.STL" scale="0.001 0.001 0.001"/>
           </geometry>
          <!-- <contact_coefficients mu="100" kp="10.0" kd="0.1"/> -->
@@ -161,5 +177,5 @@
           <origin xyz="0 0.11 0" rpy="1.57 0 0" />
           <geometry>
-            <mesh filename="package://noovelia_robot_description/meshes/Forklift model/Roues avant.STL" scale="0.001 0.001 0.001"/>
+            <mesh filename="package://forklift_description/meshes/Forklift model/Roues avant.STL" scale="0.001 0.001 0.001"/>
           </geometry>
           <material name="grey"/>
@@ -168,5 +184,5 @@
           <origin xyz="0 0.11 0" rpy="1.57 0 0" />
           <geometry>
-            <mesh filename="package://noovelia_robot_description/meshes/Forklift model/Roues avant.STL" scale="0.001 0.001 0.001"/>
+            <mesh filename="package://forklift_description/meshes/Forklift model/Roues avant.STL" scale="0.001 0.001 0.001"/>
           </geometry>
          <!-- <contact_coefficients mu="100" kp="10.0" kd="0.1"/> -->
@@ -179,4 +195,32 @@
         <!-- <axis xyz="1 0 0" /> -->
       </joint>
+   <!--Laser -->
+  <link name="laser_link">
+    <collision>
+      <origin xyz="0 0 0" rpy="0 0 0"/>
+      <geometry>
+        <box size="${laserLength} ${laserWidth} ${laserHeight}"/>
+      </geometry>
+    </collision>
+    <visual>
+      <origin xyz="0 0 0" rpy="0 0 0"/>
+      <geometry>
+        <mesh filename="package://forklift_description/meshes/Forklift model/sick_s300_laser.dae"/>
+      </geometry>
+    </visual>
+    <inertial>
+      <mass value="${laserMass}" />
+      <origin xyz="0 0 0" rpy="0 0 0"/>
+      <xacro:box_inertia
+        m="${laserMass}" x="${laserLength}" y="${laserWidth}" z="${laserHeight}"/>
+    </inertial>
+  </link>
+  <joint name="laser_joint" type="fixed">
+    <axis xyz="0 1 0" />
+    <origin xyz="${laserOffsetX} ${laserOffsetY} ${laserOffsetZ}"
+            rpy="0 0 0"/>
+    <parent link="base_link"/>
+    <child link="laser_link"/>
+  </joint>
   <!--gazebo references-->
    <gazebo reference="base_footprint">
