Commit message: Add Inertia elements. Seems like the control is much better now

File: forklift/forklift_description/urdf/forklift.xacro (robot description, xacro)
@@ -9,8 +9,12 @@
   <!--#### back/carrosserie LIFT properties ####-->
   <xacro:property name= "carrosserie_lift_width" value="1.2" />
+  <xacro:property name= "carrosserie_lift_length" value="0.7" />
+  <xacro:property name= "carrosserie_lift_height" value="1.1" />
+  <xacro:property name= "carrosserie_lift_mass" value="35" />
   <!-- Offset between link and lift mesh for proper placement-->
   <xacro:property name= "carrosserie_lift_z_offset" value="0.065" />
   <xacro:property name= "carrosserie_lift_x_offset" value="1.24" />
   <!--#### LIFT chassis/base fork properties ####-->
+  <xacro:property name= "chassis_mass" value="40" />
   <xacro:property name= "chassis_x_offset" value="0.93" />
   <xacro:property name= "chassis_y_offset" value="1.24" />
@@ -68,4 +72,16 @@
       <material name="red"/>
     </visual>
+    <inertial>
+      <mass value="${carrosserie_lift_mass}" />
+      <origin xyz="${carrosserie_lift_x_offset + carrosserie_lift_length/2}
+                   0
+                   ${carrosserie_lift_height/2}"
+              rpy="0 0 0"/>
+      <xacro:box_inertia
+        m="${carrosserie_lift_mass}"
+        x="${carrosserie_lift_width}"
+        y="${carrosserie_lift_length}"
+        z="${carrosserie_lift_height}"/>
+    </inertial>
   </link>
   <joint name="fork_joint" type="fixed">
@@ -99,9 +115,11 @@
     <inertial>
       <origin rpy="0 0 0"
-              xyz="0 0 0"/>
-      <mass value="40" />
-      <inertia ixx="0.1" ixy="0.0"
-               ixz="0.0" iyy="0.1"
-               iyz="0.0" izz="0.1" />
+              xyz="0
+                   0
+                   0.2"/>
+      <mass value="${chassis_mass}" />
+      <inertia ixx="0.08" ixy="0.0"
+               ixz="0.0" iyy="0.08"
+               iyz="0.0" izz="0.08" />
     </inertial>
   </link>

Commit message: update mass value

File: forklift/forklift_description/urdf/forklift.xacro (robot description, xacro)
@@ -126,5 +126,5 @@
   <link name="fixed_left_wheel_link">
     <inertial>
-      <mass value="0.1"/>
+      <mass value="0.2"/>
       <inertia ixx="0.01" ixy="0"
                ixz="0" iyy="0.01"
@@ -160,5 +160,5 @@
   <link name="fixed_right_wheel_link">
     <inertial>
-      <mass value="0.1"/>
+      <mass value="0.2"/>
       <inertia ixx="0.01" ixy="0"
                ixz="0" iyy="0.01"

Commit message: add nav sensor

File: forklift/forklift_description/urdf/forklift.xacro (robot description, xacro)
@@ -20,9 +20,17 @@
   <xacro:property name= "chassis_y_offset" value="1.24" />
   <xacro:property name= "chassis_z_offset" value="0.28" />
-  <!--### main wheel properties that performs steer + move ####-->
+  <!--#### main wheel properties that performs steer + move ####-->
   <xacro:property name="wheel_width" value="0.08" />
   <xacro:property name="wheel_radius" value="0.10" />
   <xacro:property name="wheel_mass" value="10" /> <!-- in kg-->
   <xacro:property name="wheel_x_offset" value="1.7" /> <!-- in kg-->
+  <!--#### Navigation Laser properties ####-->
+	<xacro:property name="laser_mass" value="0.01"/>
+	<xacro:property name="laser_length" value="0.05"/>
+	<xacro:property name="laser_width" value="0.05"/>
+	<xacro:property name="laser_height" value="0.07"/>
+	<xacro:property name="laser_offset_x" value="0.75"/>
+  <xacro:property name="laser_offset_y" value="0"/>
+	<xacro:property name="laser_offset_z" value="2.8"/>
   <!--### caster/fixed wheel properties ####-->
   <xacro:property name="caster_radius" value="0.06" />
@@ -246,4 +254,37 @@
     <origin xyz="0 0 0" rpy="0 0 0" />
     <axis xyz="0 1 0" />
+  </joint>
+   <!--Navigation Laser -->
+  <link name="laser_link">
+    <collision>
+      <origin xyz="0 0 0"
+              rpy="0 0 0"/>
+      <geometry>
+        <box size="${laser_length} ${laser_width} ${laser_height}"/>
+      </geometry>
+    </collision>
+    <visual>
+      <origin xyz="0 0 0"
+              rpy="0 0 0"/>
+      <geometry>
+        <mesh filename="package://forklift_description/meshes/Forklift model/sick_s300_laser.dae"/>
+      </geometry>
+    </visual>
+    <inertial>
+      <mass value="${laser_mass}" />
+      <origin xyz="0 0 0" rpy="0 0 0"/>
+      <xacro:box_inertia
+        m = "${laser_mass}"
+        x = "${laser_length}"
+        y = "${laser_width}"
+        z = "${laser_height}"/>
+    </inertial>
+  </link>
+  <joint name="laser_joint" type="fixed">
+    <axis xyz="0 1 0" />
+    <origin xyz="${laser_offset_x} ${laser_offset_y} ${laser_offset_z}"
+            rpy="0 0 0"/>
+    <parent link="base_link"/>
+    <child link="laser_link"/>
   </joint>
  <!--#### GAZEBO references ####-->
@@ -312,3 +353,41 @@
     </plugin>
   </gazebo>
+ <gazebo reference="laser_link">
+    <!-- Don't use type="gpu_ray" -->
+    <sensor type="ray"
+            name="nav_sensor">
+      <pose>0 0 0 0 0 0</pose>
+      <visualize>false</visualize>
+      <update_rate>40</update_rate>
+      <ray>
+        <scan>
+          <horizontal>
+            <samples>720</samples>
+            <resolution>1</resolution>
+            <min_angle>-3.1415926</min_angle>
+            <max_angle>3.1415926</max_angle>
+          </horizontal>
+        </scan>
+        <range>
+          <min>0.10</min>
+          <max>30.0</max>
+          <resolution>0.01</resolution>
+        </range>
+        <noise>
+          <type>gaussian</type>
+          <!-- Noise parameters based on published spec for Hokuyo laser
+               achieving "+-30mm" accuracy at range < 10m.  A mean of 0.0m and
+               stddev of 0.01m will put 99.7% of samples within 0.03m of the true
+               reading. -->
+          <mean>0.0</mean>
+          <stddev>0.01</stddev>
+        </noise>
+      </ray>
+        <plugin name="gazebo_ros_laser_controller"
+              filename="libgazebo_ros_laser.so">
+        <topicName>/laser/scan</topicName>
+        <frameName>laser_link</frameName>
+      </plugin>
+    </sensor>
+  </gazebo>
 </robot>

Commit message: initial code base for gmapping

File: forklift/forklift_description/urdf/forklift.xacro (robot description, xacro)
@@ -1,4 +1,5 @@
 <?xml version="1.0" ?>
-<robot name="noovelia_forklift" xmlns:xacro="http://www.ros.org/wiki/xacro">
+<robot name="noovelia_forklift"
+  xmlns:xacro="http://www.ros.org/wiki/xacro">
   <xacro:include filename="$(find forklift_description)/urdf/material.xacro" />
   <!--#### various constants ####-->
@@ -23,14 +24,16 @@
   <xacro:property name="wheel_width" value="0.08" />
   <xacro:property name="wheel_radius" value="0.10" />
-  <xacro:property name="wheel_mass" value="10" /> <!-- in kg-->
-  <xacro:property name="wheel_x_offset" value="1.7" /> <!-- in kg-->
+  <xacro:property name="wheel_mass" value="10" />
+  <!-- in kg-->
+  <xacro:property name="wheel_x_offset" value="1.7" />
+  <!-- in kg-->
   <!--#### Navigation Laser properties ####-->
-	<xacro:property name="laser_mass" value="0.01"/>
-	<xacro:property name="laser_length" value="0.05"/>
-	<xacro:property name="laser_width" value="0.05"/>
-	<xacro:property name="laser_height" value="0.07"/>
-	<xacro:property name="laser_offset_x" value="0.75"/>
+  <xacro:property name="laser_mass" value="0.01"/>
+  <xacro:property name="laser_length" value="0.05"/>
+  <xacro:property name="laser_width" value="0.05"/>
+  <xacro:property name="laser_height" value="0.07"/>
+  <xacro:property name="laser_offset_x" value="0.75"/>
   <xacro:property name="laser_offset_y" value="0"/>
-	<xacro:property name="laser_offset_z" value="2.8"/>
+  <xacro:property name="laser_offset_z" value="2.8"/>
   <!--### caster/fixed wheel properties ####-->
   <xacro:property name="caster_radius" value="0.06" />
@@ -39,13 +42,8 @@
   <!--#### Intertia Elements of various objects and shapes ####-->
   <xacro:macro name="cylinder_inertia" params="m r h">
-      <inertia  ixx="${m*(3*r*r+h*h)/12}" ixy = "0" ixz = "0"
-                iyy="${m*(3*r*r+h*h)/12}" iyz = "0"
-                izz="${m*r*r/2}" />
+    <inertia ixx="${m*(3*r*r+h*h)/12}" ixy = "0" ixz = "0" iyy="${m*(3*r*r+h*h)/12}" iyz = "0" izz="${m*r*r/2}" />
   </xacro:macro>
   <xacro:macro name="box_inertia" params="m x y z">
-    <inertia  ixx="${m*(y*y+z*z)/12}" ixy = "0" ixz = "0"
-    			iyy="${m*(x*x+z*z)/12}" iyz = "0"
-    			izz="${m*(x*x+z*z)/12}"
-  />
+    <inertia ixx="${m*(y*y+z*z)/12}" ixy = "0" ixz = "0" iyy="${m*(x*x+z*z)/12}" iyz = "0" izz="${m*(x*x+z*z)/12}" />
   </xacro:macro>
   <!--#### Links and Joints of Forklift ####-->
@@ -53,6 +51,5 @@
   </link>
   <joint name="base_footprint_joint" type="fixed">
-    <origin xyz="0 0 ${caster_radius}"
-            rpy="0 0 0" />
+    <origin xyz="0 0 ${caster_radius}" rpy="0 0 0" />
     <child link="base_link" />
     <parent link="base_footprint"/>
@@ -60,21 +57,17 @@
   <link name="base_link">
     <collision name="base_link_collision">
-      <origin rpy="${M_PI_2} 0 ${M_PI_2}"
-              xyz="${carrosserie_lift_x_offset}
+      <origin rpy="${M_PI_2} 0 ${M_PI_2}" xyz="${carrosserie_lift_x_offset}
                   -${carrosserie_lift_width/2}
                   -${carrosserie_lift_z_offset}"/>
       <geometry>
-        <mesh filename="package://forklift_description/meshes/Forklift model/carrosserie lift.STL"
-              scale="0.001 0.001 0.001"/>
+        <mesh filename="package://forklift_description/meshes/Forklift model/carrosserie lift.STL" scale="0.001 0.001 0.001"/>
       </geometry>
     </collision>
     <visual name="base_link_visual">
-      <origin rpy="${M_PI_2} 0 ${M_PI_2}"
-              xyz="${carrosserie_lift_x_offset}
+      <origin rpy="${M_PI_2} 0 ${M_PI_2}" xyz="${carrosserie_lift_x_offset}
                   -${carrosserie_lift_width/2}
                   -${carrosserie_lift_z_offset}"/>
       <geometry>
-        <mesh filename="package://forklift_description/meshes/Forklift model/carrosserie lift.STL"
-              scale="0.001 0.001 0.001"/>
+        <mesh filename="package://forklift_description/meshes/Forklift model/carrosserie lift.STL" scale="0.001 0.001 0.001"/>
       </geometry>
       <material name="red"/>
@@ -84,16 +77,10 @@
       <origin xyz="${carrosserie_lift_x_offset + carrosserie_lift_length/2}
                    0
-                   0.1"
-              rpy="0 0 0"/>
-      <xacro:box_inertia
-        m="${carrosserie_lift_mass}"
-        x="${carrosserie_lift_width}"
-        y="${carrosserie_lift_length}"
-        z="${carrosserie_lift_height}"/>
+                   0.1" rpy="0 0 0"/>
+      <xacro:box_inertia m="${carrosserie_lift_mass}" x="${carrosserie_lift_width}" y="${carrosserie_lift_length}" z="${carrosserie_lift_height}"/>
     </inertial>
   </link>
   <joint name="fork_joint" type="fixed">
-    <origin xyz="0.18 0.0 0.0"
-            rpy="0 0 0" />
+    <origin xyz="0.18 0.0 0.0" rpy="0 0 0" />
     <parent link="base_link" />
     <child link="base_fork"/>
@@ -101,33 +88,26 @@
   <link name="base_fork">
     <collision name="fork_collision">
-      <origin rpy="${M_PI_2} 0 ${M_PI_2}"
-              xyz="-${chassis_x_offset}
+      <origin rpy="${M_PI_2} 0 ${M_PI_2}" xyz="-${chassis_x_offset}
                    -${chassis_y_offset}
                    -${chassis_z_offset}"/>
       <geometry>
-        <mesh filename="package://forklift_description/meshes/Forklift model/chassis AGV FL.STL"
-              scale="0.001 0.001 0.001"/>
+        <mesh filename="package://forklift_description/meshes/Forklift model/chassis AGV FL.STL" scale="0.001 0.001 0.001"/>
       </geometry>
     </collision>
     <visual name="fork_visual">
-      <origin rpy="${M_PI_2} 0 ${M_PI_2}"
-              xyz="-${chassis_x_offset}
+      <origin rpy="${M_PI_2} 0 ${M_PI_2}" xyz="-${chassis_x_offset}
                    -${chassis_y_offset}
                    -${chassis_z_offset}"/>
       <geometry>
-        <mesh filename="package://forklift_description/meshes/Forklift model/chassis AGV FL.STL"
-              scale="0.001 0.001 0.001"/>
+        <mesh filename="package://forklift_description/meshes/Forklift model/chassis AGV FL.STL" scale="0.001 0.001 0.001"/>
       </geometry>
       <material name="white"/>
     </visual>
     <inertial>
-      <origin rpy="0 0 0"
-              xyz="0
+      <origin rpy="0 0 0" xyz="0
                    0
                    0.2"/>
       <mass value="${chassis_mass}" />
-      <inertia ixx="0.08" ixy="0.0"
-               ixz="0.0" iyy="0.08"
-               iyz="0.0" izz="0.08" />
+      <inertia ixx="0.08" ixy="0.0" ixz="0.0" iyy="0.08" iyz="0.0" izz="0.08" />
     </inertial>
   </link>
@@ -135,77 +115,61 @@
     <inertial>
       <mass value="0.2"/>
-      <inertia ixx="0.01" ixy="0"
-               ixz="0" iyy="0.01"
-               iyz="0" izz="0.01" />
+      <inertia ixx="0.01" ixy="0" ixz="0" iyy="0.01" iyz="0" izz="0.01" />
       <origin/>
     </inertial>
     <visual name="fixed_left_wheel_visual">
-      <origin xyz="0 0 0"
-              rpy="${M_PI_2} 0 0" />
-      <geometry>
-        <cylinder radius="${caster_radius}"
-                  length="${caster_length}" />
+      <origin xyz="0 0 0" rpy="${M_PI_2} 0 0" />
+      <geometry>
+        <cylinder radius="${caster_radius}" length="${caster_length}" />
       </geometry>
       <material name="grey"/>
     </visual>
     <collision name="fixed_left_wheel_collision">
-      <origin xyz="0 0 0"
-              rpy="${M_PI_2} 0 0" />
-      <geometry>
-        <cylinder radius="${caster_radius}"
-                  length="${caster_length}" />
+      <origin xyz="0 0 0" rpy="${M_PI_2} 0 0" />
+      <geometry>
+        <cylinder radius="${caster_radius}" length="${caster_length}" />
       </geometry>
       <!-- <contact_coefficients mu="100" kp="10.0" kd="0.1"/> -->
     </collision>
   </link>
-  <joint name="base2fixed_left_wheel_joint" type="continuous">
+  <joint name="base2fixed_left_wheel_joint" type="fixed">
     <parent link="base_link"/>
     <child link="fixed_left_wheel_link"/>
-    <origin xyz="0 ${caster_y_offset} 0"
-            rpy="0 0 0" />
-    <axis xyz="0 1 0" />
+    <origin xyz="0 ${caster_y_offset} 0" rpy="0 0 0" />
+    <!-- <axis xyz="0 1 0" /> -->
   </joint>
   <link name="fixed_right_wheel_link">
     <inertial>
       <mass value="0.2"/>
-      <inertia ixx="0.01" ixy="0"
-               ixz="0" iyy="0.01"
-               iyz="0" izz="0.01" />
+      <inertia ixx="0.01" ixy="0" ixz="0" iyy="0.01" iyz="0" izz="0.01" />
       <origin/>
     </inertial>
     <visual>
-      <origin xyz="0 0 0"
-              rpy="${M_PI_2} 0 0" />
-      <geometry>
-        <cylinder radius="${caster_radius}"
-                  length="${caster_length}" />
+      <origin xyz="0 0 0" rpy="${M_PI_2} 0 0" />
+      <geometry>
+        <cylinder radius="${caster_radius}" length="${caster_length}" />
       </geometry>
       <material name="grey"/>
     </visual>
     <collision>
-      <origin xyz="0 0 0"
-              rpy="${M_PI_2} 0 0" />
-      <geometry>
-        <cylinder radius="${caster_radius}"
-                  length="${caster_length}" />
+      <origin xyz="0 0 0" rpy="${M_PI_2} 0 0" />
+      <geometry>
+        <cylinder radius="${caster_radius}" length="${caster_length}" />
       </geometry>
       <!-- <contact_coefficients mu="100" kp="10.0" kd="0.1"/> -->
     </collision>
   </link>
-  <joint name="base2fixed_right_wheel_joint" type="continuous">
+  <joint name="base2fixed_right_wheel_joint" type="fixed">
     <parent link="base_link"/>
     <child link="fixed_right_wheel_link"/>
-    <origin xyz="0 -${caster_y_offset} 0"
-            rpy="0 0 0" />
-    <axis xyz="0 1 0" />
+    <origin xyz="0 -${caster_y_offset} 0" rpy="0 0 0" />
+    <!-- <axis xyz="0 1 0" /> -->
   </joint>
   <link name="steer_link">
     <inertial>
       <mass value="0.01"/>
-      <inertia ixx="0.001" ixy="0"
-               ixz="0" iyy="0.001"
-               iyz="0" izz="0.001" />
+      <inertia ixx="0.001" ixy="0" ixz="0" iyy="0.001" iyz="0" izz="0.001" />
       <origin/>
-      </inertial>
+    </inertial>
     <visual>
       <origin xyz="0 0 0" rpy="0 0 0" />
@@ -219,7 +183,5 @@
     <inertial>
       <mass value="10"/>
-      <inertia ixx="0.01" ixy="0"
-               ixz="0" iyy="0.01"
-               iyz="0" izz="0.01" />
+      <inertia ixx="0.01" ixy="0" ixz="0" iyy="0.01" iyz="0" izz="0.01" />
       <origin/>
     </inertial>
@@ -227,15 +189,12 @@
       <origin xyz="0 0 0" rpy="${M_PI_2} 0 0" />
       <geometry>
-        <cylinder radius="${wheel_radius}"
-                  length="${wheel_width}" />
+        <cylinder radius="${wheel_radius}" length="${wheel_width}" />
       </geometry>
       <material name="black"/>
     </visual>
     <collision>
-      <origin xyz="0 0 0"
-              rpy="${M_PI_2} 0 0" />
-      <geometry>
-        <cylinder radius="${wheel_radius}"
-                  length="${wheel_width}" />
+      <origin xyz="0 0 0" rpy="${M_PI_2} 0 0" />
+      <geometry>
+        <cylinder radius="${wheel_radius}" length="${wheel_width}" />
       </geometry>
     </collision>
@@ -255,9 +214,8 @@
     <axis xyz="0 1 0" />
   </joint>
-   <!--Navigation Laser -->
+  <!--Navigation Laser -->
   <link name="laser_link">
     <collision>
-      <origin xyz="0 0 0"
-              rpy="0 0 0"/>
+      <origin xyz="0 0 0" rpy="0 0 0"/>
       <geometry>
         <box size="${laser_length} ${laser_width} ${laser_height}"/>
@@ -265,6 +223,5 @@
     </collision>
     <visual>
-      <origin xyz="0 0 0"
-              rpy="0 0 0"/>
+      <origin xyz="0 0 0" rpy="0 0 0"/>
       <geometry>
         <mesh filename="package://forklift_description/meshes/Forklift model/sick_s300_laser.dae"/>
@@ -283,10 +240,9 @@
   <joint name="laser_joint" type="fixed">
     <axis xyz="0 1 0" />
-    <origin xyz="${laser_offset_x} ${laser_offset_y} ${laser_offset_z}"
-            rpy="0 0 0"/>
+    <origin xyz="${laser_offset_x} ${laser_offset_y} ${laser_offset_z}" rpy="0 0 0"/>
     <parent link="base_link"/>
     <child link="laser_link"/>
   </joint>
- <!--#### GAZEBO references ####-->
+  <!--#### GAZEBO references ####-->
   <gazebo reference="base_footprint">
     <turnGravityOff>false</turnGravityOff>
@@ -303,32 +259,32 @@
     <material>Gazebo/Blue</material>
   </gazebo>
-  <gazebo reference="fixed_left_wheel_link" >
+  <gazebo reference="fixed_left_wheel_link">
     <!-- <mu1 value="10000.0" />
     <mu2 value="10000.0" />
-    <kp  value="10000000000.0" />
-    <kd  value="1.0" /> -->
+    <kp value="10000000000.0" />
+    <kd value="1.0" /> -->
     <material>Gazebo/Black</material>
   </gazebo>
-  <gazebo reference="fixed_right_wheel_link" >
+  <gazebo reference="fixed_right_wheel_link">
     <!-- <mu1 value="10000.0" />
     <mu2 value="10000.0" />
-    <kp  value="10000000000.0" />
-    <kd  value="1.0" /> -->
+    <kp value="10000000000.0" />
+    <kd value="1.0" /> -->
     <material>Gazebo/Black</material>
   </gazebo>
-  <gazebo reference="sd_wheel_link" >
+  <gazebo reference="sd_wheel_link">
     <mu1 value="10000.0" />
     <mu2 value="10000.0" />
-    <kp  value="10000000000.0" />
-    <kd  value="1.0" />
-  <material>Gazebo/Black</material>
+    <kp value="10000000000.0" />
+    <kd value="1.0" />
+    <material>Gazebo/Black</material>
   </gazebo>
   <!-- ros_control plugin -->
   <gazebo>
     <plugin name="gazebo_ros_control" filename="libgazebo_ros_control.so">
-<!--      <robotNamespace>/forklift</robotNamespace> -->
+      <!--      <robotNamespace>/forklift</robotNamespace> -->
     </plugin>
   </gazebo>
-   <gazebo>
+  <gazebo>
     <plugin name="steer_drive_controller" filename="libgazebo_ros_steer_drive.so">
       <alwaysOn>true</alwaysOn>
@@ -353,8 +309,7 @@
     </plugin>
   </gazebo>
- <gazebo reference="laser_link">
+  <gazebo reference="laser_link">
     <!-- Don't use type="gpu_ray" -->
-    <sensor type="ray"
-            name="nav_sensor">
+    <sensor type="ray" name="nav_sensor">
       <pose>0 0 0 0 0 0</pose>
       <visualize>false</visualize>
@@ -384,6 +339,5 @@
         </noise>
       </ray>
-        <plugin name="gazebo_ros_laser_controller"
-              filename="libgazebo_ros_laser.so">
+      <plugin name="gazebo_ros_laser_controller" filename="libgazebo_ros_laser.so">
         <topicName>/laser/scan</topicName>
         <frameName>laser_link</frameName>

Commit message: added one laser in the bottom

File: forklift/forklift_description/urdf/forklift.xacro (robot description, xacro)
@@ -23,5 +23,5 @@
   <!--#### main wheel properties that performs steer + move ####-->
   <xacro:property name="wheel_width" value="0.08" />
-  <xacro:property name="wheel_radius" value="0.10" />
+  <xacro:property name="wheel_radius" value="0.12" />
   <xacro:property name="wheel_mass" value="10" />
   <!-- in kg-->
@@ -30,12 +30,12 @@
   <!--#### Navigation Laser properties ####-->
   <xacro:property name="laser_mass" value="0.01"/>
-  <xacro:property name="laser_length" value="0.05"/>
-  <xacro:property name="laser_width" value="0.05"/>
-  <xacro:property name="laser_height" value="0.07"/>
-  <xacro:property name="laser_offset_x" value="0.75"/>
-  <xacro:property name="laser_offset_y" value="0"/>
-  <xacro:property name="laser_offset_z" value="2.8"/>
+  <xacro:property name="laser_length" value="0.08"/>
+  <xacro:property name="laser_width" value="0.07"/>
+  <xacro:property name="laser_height" value="0.06"/>
+  <xacro:property name="laser_offset_x" value="0.25"/>
+  <xacro:property name="laser_offset_y" value="0.45"/>
+  <xacro:property name="laser_offset_z" value="${laser_height/2}"/>
   <!--### caster/fixed wheel properties ####-->
-  <xacro:property name="caster_radius" value="0.06" />
+  <xacro:property name="caster_radius" value="0.08" />
   <xacro:property name="caster_length" value="0.16" />
   <xacro:property name="caster_y_offset" value="0.52" />
@@ -225,5 +225,5 @@
       <origin xyz="0 0 0" rpy="0 0 0"/>
       <geometry>
-        <mesh filename="package://forklift_description/meshes/Forklift model/sick_s300_laser.dae"/>
+        <box size="${laser_length} ${laser_width} ${laser_height}"/>
       </geometry>
     </visual>
@@ -240,6 +240,6 @@
   <joint name="laser_joint" type="fixed">
     <axis xyz="0 1 0" />
-    <origin xyz="${laser_offset_x} ${laser_offset_y} ${laser_offset_z}" rpy="0 0 0"/>
-    <parent link="base_link"/>
+    <origin xyz="${laser_offset_x} ${laser_offset_y} -${laser_offset_z}" rpy="0 0 0"/>
+    <parent link="steer_link"/>
     <child link="laser_link"/>
   </joint>
