Commit message: Added Nav1 laser in separate xacro

File: forklift/forklift_description/urdf/forklift.xacro (robot description, xacro)
@@ -214,34 +214,7 @@
     <axis xyz="0 1 0" />
   </joint>
-  <!--Navigation Laser -->
-  <link name="laser_link">
-    <collision>
-      <origin xyz="0 0 0" rpy="0 0 0"/>
-      <geometry>
-        <box size="${laser_length} ${laser_width} ${laser_height}"/>
-      </geometry>
-    </collision>
-    <visual>
-      <origin xyz="0 0 0" rpy="0 0 0"/>
-      <geometry>
-        <box size="${laser_length} ${laser_width} ${laser_height}"/>
-      </geometry>
-    </visual>
-    <inertial>
-      <mass value="${laser_mass}" />
-      <origin xyz="0 0 0" rpy="0 0 0"/>
-      <xacro:box_inertia
-        m = "${laser_mass}"
-        x = "${laser_length}"
-        y = "${laser_width}"
-        z = "${laser_height}"/>
-    </inertial>
-  </link>
-  <joint name="laser_joint" type="fixed">
-    <axis xyz="0 1 0" />
-    <origin xyz="${laser_offset_x} ${laser_offset_y} -${laser_offset_z}" rpy="0 0 0"/>
-    <parent link="steer_link"/>
-    <child link="laser_link"/>
-  </joint>
+  <!--#### Laser####-->
+  <xacro:include filename="$(find forklift_description)/urdf/laser.xacro" />
+  <xacro:laser name = "nav1" x_offset = "${laser_offset_x}" y_offset = "${laser_offset_y}" z_offset = "${laser_offset_z}"/>
   <!--#### GAZEBO references ####-->
   <gazebo reference="base_footprint">
@@ -310,39 +283,3 @@
     </plugin>
   </gazebo>
-  <gazebo reference="laser_link">
-    <!-- Don't use type="gpu_ray" -->
-    <sensor type="ray" name="nav_sensor">
-      <pose>0 0 0 0 0 0</pose>
-      <visualize>false</visualize>
-      <update_rate>40</update_rate>
-      <ray>
-        <scan>
-          <horizontal>
-            <samples>720</samples>
-            <resolution>1</resolution>
-            <min_angle>-3.1415926</min_angle>
-            <max_angle>3.1415926</max_angle>
-          </horizontal>
-        </scan>
-        <range>
-          <min>0.10</min>
-          <max>30.0</max>
-          <resolution>0.01</resolution>
-        </range>
-        <noise>
-          <type>gaussian</type>
-          <!-- Noise parameters based on published spec for Hokuyo laser
-               achieving "+-30mm" accuracy at range < 10m.  A mean of 0.0m and
-               stddev of 0.01m will put 99.7% of samples within 0.03m of the true
-               reading. -->
-          <mean>0.0</mean>
-          <stddev>0.01</stddev>
-        </noise>
-      </ray>
-      <plugin name="gazebo_ros_laser_controller" filename="libgazebo_ros_laser.so">
-        <topicName>/laser/scan</topicName>
-        <frameName>laser_link</frameName>
-      </plugin>
-    </sensor>
-  </gazebo>
 </robot>

File: forklift/forklift_description/urdf/laser.xacro (robot description, xacro)
@@ -1,5 +1,71 @@
 <?xml version="1.0"?>
 <robot xmlns:xacro="http://www.ros.org/wiki/xacro">
-    <xacro:macro name="laser">
+    <xacro:macro name="laser" params="name x_offset y_offset z_offset">
+        <!--Navigation Laser -->
+        <link name="${name}_laser_link">
+            <collision>
+                <origin xyz="0 0 0" rpy="0 0 0"/>
+                <geometry>
+                    <box size="${laser_length} ${laser_width} ${laser_height}"/>
+                </geometry>
+            </collision>
+            <visual>
+                <origin xyz="0 0 0" rpy="0 0 0"/>
+                <geometry>
+                    <box size="${laser_length} ${laser_width} ${laser_height}"/>
+                </geometry>
+            </visual>
+            <inertial>
+                <mass value="${laser_mass}" />
+                <origin xyz="0 0 0" rpy="0 0 0"/>
+                <xacro:box_inertia
+                    m = "${laser_mass}"
+                    x = "${laser_length}"
+                    y = "${laser_width}"
+                    z = "${laser_height}"/>
+            </inertial>
+        </link>
+        <joint name="laser_joint" type="fixed">
+            <axis xyz="0 1 0" />
+            <origin xyz="${x_offset} ${y_offset} -${z_offset}" rpy="0 0 0"/>
+            <parent link="steer_link"/>
+            <child link="${name}_laser_link"/>
+        </joint>
+        <gazebo reference="${name}_laser_link">
+            <!-- Don't use type="gpu_ray" -->
+            <sensor type="ray" name="nav_sensor">
+                <pose>0 0 0 0 0 0</pose>
+                <visualize>false</visualize>
+                <update_rate>40</update_rate>
+                <ray>
+                    <scan>
+                        <horizontal>
+                            <samples>720</samples>
+                            <resolution>1</resolution>
+                            <min_angle>-3.1415926</min_angle>
+                            <max_angle>3.1415926</max_angle>
+                        </horizontal>
+                    </scan>
+                    <range>
+                        <min>0.10</min>
+                        <max>30.0</max>
+                        <resolution>0.01</resolution>
+                    </range>
+                    <noise>
+                        <type>gaussian</type>
+                        <!-- Noise parameters based on published spec for Hokuyo laser
+                        achieving "+-30mm" accuracy at range < 10m.  A mean of 0.0m and
+                        stddev of 0.01m will put 99.7% of samples within 0.03m of the true
+                        reading. -->
+                        <mean>0.0</mean>
+                        <stddev>0.01</stddev>
+                    </noise>
+                </ray>
+                <plugin name="gazebo_ros_laser_controller" filename="libgazebo_ros_laser.so">
+                    <topicName>${name}/laser/scan</topicName>
+                    <frameName>${name}_laser_link</frameName>
+                </plugin>
+            </sensor>
+        </gazebo>
     </xacro:macro>
 </robot>

Commit message: added all three lasers

File: forklift/forklift_description/urdf/forklift.xacro (robot description, xacro)
@@ -33,6 +33,4 @@
   <xacro:property name="laser_width" value="0.07"/>
   <xacro:property name="laser_height" value="0.06"/>
-  <xacro:property name="laser_offset_x" value="0.25"/>
-  <xacro:property name="laser_offset_y" value="0.45"/>
   <xacro:property name="laser_offset_z" value="${laser_height/2}"/>
   <!--### caster/fixed wheel properties ####-->
@@ -216,5 +214,7 @@
   <!--#### Laser####-->
   <xacro:include filename="$(find forklift_description)/urdf/laser.xacro" />
-  <xacro:laser name = "nav1" x_offset = "${laser_offset_x}" y_offset = "${laser_offset_y}" z_offset = "${laser_offset_z}"/>
+  <xacro:laser name = "nav1" x_offset = "1.7" y_offset = "0.55" z_offset = "${laser_offset_z}"/>
+  <xacro:laser name = "nav2" x_offset = "1.7" y_offset = "-0.55" z_offset = "${laser_offset_z}"/>
+  <xacro:laser name = "nav3" x_offset = "0.5" y_offset = "0" z_offset = "${laser_offset_z}"/>
   <!--#### GAZEBO references ####-->
   <gazebo reference="base_footprint">

File: forklift/forklift_description/urdf/laser.xacro (robot description, xacro)
@@ -26,8 +26,8 @@
             </inertial>
         </link>
-        <joint name="laser_joint" type="fixed">
+        <joint name="${name}_laser_joint" type="fixed">
             <axis xyz="0 1 0" />
             <origin xyz="${x_offset} ${y_offset} -${z_offset}" rpy="0 0 0"/>
-            <parent link="steer_link"/>
+            <parent link="base_fork"/>
             <child link="${name}_laser_link"/>
         </joint>

Commit message: Formatting

File: forklift/forklift_description/urdf/forklift.xacro (robot description, xacro)
@@ -214,7 +214,7 @@
   <!--#### Laser####-->
   <xacro:include filename="$(find forklift_description)/urdf/laser.xacro" />
-  <xacro:laser name = "nav1" x_offset = "1.7" y_offset = "0.55" z_offset = "${laser_offset_z}"/>
-  <xacro:laser name = "nav2" x_offset = "1.7" y_offset = "-0.55" z_offset = "${laser_offset_z}"/>
-  <xacro:laser name = "nav3" x_offset = "0.5" y_offset = "0" z_offset = "${laser_offset_z}"/>
+  <xacro:laser name = "nav1" x_offset = "1.7" y_offset = "0.55" z_offset = "${laser_offset_z}" yaw = "0"/>
+  <xacro:laser name = "nav2" x_offset = "1.7" y_offset = "-0.55" z_offset = "${laser_offset_z}" yaw = "0"/>
+  <xacro:laser name = "nav3" x_offset = "0.5" y_offset = "0" z_offset = "${laser_offset_z}" yaw = "${M_PI}"/>
   <!--#### GAZEBO references ####-->
   <gazebo reference="base_footprint">

File: forklift/forklift_description/urdf/laser.xacro (robot description, xacro)
@@ -1,5 +1,5 @@
 <?xml version="1.0"?>
 <robot xmlns:xacro="http://www.ros.org/wiki/xacro">
-    <xacro:macro name="laser" params="name x_offset y_offset z_offset">
+    <xacro:macro name="laser" params="name x_offset y_offset z_offset yaw">
         <!--Navigation Laser -->
         <link name="${name}_laser_link">
@@ -28,5 +28,5 @@
         <joint name="${name}_laser_joint" type="fixed">
             <axis xyz="0 1 0" />
-            <origin xyz="${x_offset} ${y_offset} -${z_offset}" rpy="0 0 0"/>
+            <origin xyz="${x_offset} ${y_offset} -${z_offset}" rpy="0 0 ${yaw}"/>
             <parent link="base_fork"/>
             <child link="${name}_laser_link"/>
@@ -34,5 +34,5 @@
         <gazebo reference="${name}_laser_link">
             <!-- Don't use type="gpu_ray" -->
-            <sensor type="ray" name="nav_sensor">
+            <sensor type="ray" name="${name}_sensor">
                 <pose>0 0 0 0 0 0</pose>
                 <visualize>false</visualize>
